Commit message: Multi-robot: namespaced spawn, frame prefixes, serial goal driver
Stock nav2 (MPPI) throughout; nothing uses mpc_control/acados.

- xacros take prefix/ns args: every link, joint, TF frame and Gazebo topic is
  per-robot. Single robot (both empty) generates the original names unchanged.
- multi_gazebo.launch.py spawns N namespaced robots, staggered, and bridges
  /clock, which multiple stacks need.
- multi_nav2.launch.py rewrites nav.yaml per robot (absolute topics and bare
  frames) so nav.yaml stays the single source of truth. Localization is a
  static identity map->rX/odom, since gz odometry is world-absolute.
- navigation.launch.py was missing PushROSNamespace, so its namespace arg only
  reached RewrittenYaml and all robots' nodes collided in the root namespace.
- DiffDrive no longer publishes odom/TF; the odometry plugin was already doing
  it, so the two raced on the same topic.
- Sensors system plugin moved from lidar.xacro to the world, so it loads once
  rather than once per robot. Lidar samples now an arg (3600 -> 720 for N robots).
- serial_driver drives one robot at a time to completion, then the next.

File: src/nav2_mobile_robot/urdf/gazebo_control.xacro (robot description, xacro)
@@ -5,22 +5,24 @@
   <gazebo>
     <plugin filename="gz-sim-diff-drive-system" name="gz::sim::systems::DiffDrive">
-      <left_joint>left_wheel_joint</left_joint>
-      <right_joint>right_wheel_joint</right_joint>
+      <left_joint>${prefix}left_wheel_joint</left_joint>
+      <right_joint>${prefix}right_wheel_joint</right_joint>
       <wheel_separation>${2*base_radius}</wheel_separation>
       <wheel_radius>${wheel_radius}</wheel_radius>
-      <frame_id>odom</frame_id>
-      <child_frame_id>base_link</child_frame_id>
-      <publish_odom>true</publish_odom>
-      <publish_odom_tf>true</publish_odom_tf>
-      <odom_publish_frequency>10</odom_publish_frequency>
-      <topic>cmd_vel</topic>
-      <robotBaseFrame>base_link</robotBaseFrame>
+      <frame_id>${prefix}odom</frame_id>
+      <child_frame_id>${prefix}base_link</child_frame_id>
+      <!-- Odometry comes from gz-sim-odometry-publisher-system (odom_plugin.xacro)
+           at 50 Hz. DiffDrive must NOT also publish, or two publishers race on
+           the same topic and TF. DiffDrive here only actuates the wheels. -->
+      <publish_odom>false</publish_odom>
+      <publish_odom_tf>false</publish_odom_tf>
+      <topic>${ns}/cmd_vel</topic>
+      <robotBaseFrame>${prefix}base_link</robotBaseFrame>
     </plugin>
   </gazebo>
-  <gazebo reference="passive_wheel_front_link">
+  <gazebo reference="${prefix}passive_wheel_front_link">
     <mu1 value="0.1" />
     <mu2 value="0.1" />
   </gazebo>
-  <gazebo reference="passive_wheel_back_link">
+  <gazebo reference="${prefix}passive_wheel_back_link">
     <mu1 value="0.1" />
     <mu2 value="0.1" />
@@ -28,7 +30,7 @@
   <gazebo>
     <plugin filename="gz-sim-joint-state-publisher-system" name="gz::sim::systems::JointStatePublisher">
-      <topic>/joint_states</topic>
-      <joint_name>left_wheel_joint</joint_name>
-      <joint_name>right_wheel_joint</joint_name>
+      <topic>${ns}/joint_states</topic>
+      <joint_name>${prefix}left_wheel_joint</joint_name>
+      <joint_name>${prefix}right_wheel_joint</joint_name>
     </plugin>
   </gazebo>

File: src/nav2_mobile_robot/urdf/lidar.xacro (robot description, xacro)
@@ -3,5 +3,9 @@
   xmlns:xacro="http://ros.org/wiki/xacro">
   <xacro:property name="PI" value="3.14159"/>
-  <link name="lidar_link">
+  <!-- 3600 samples (0.1 deg) is what a single robot uses so adjacent rays stay
+       inside one 0.003125 m map cell out to ~1.8 m. With N robots the GPU lidar
+       cost multiplies, so the multi-robot launch lowers this. -->
+  <xacro:arg name="lidar_samples" default="3600" />
+  <link name="${prefix}lidar_link">
     <visual>
       <origin xyz="0 0 0.05" rpy="0 0 0"/>
@@ -22,19 +26,17 @@
     </inertial>
   </link>
-  <joint name='lidar_sensor_joint' type='fixed'>
-    <parent link="base_link"/>
-    <child link="lidar_link"/>
+  <joint name='${prefix}lidar_sensor_joint' type='fixed'>
+    <parent link="${prefix}base_link"/>
+    <child link="${prefix}lidar_link"/>
   </joint>
-  <gazebo reference="lidar_link">
+  <gazebo reference="${prefix}lidar_link">
     <sensor name="lidar" type='gpu_lidar'>
       <pose>0 0 0.2 0 0 0</pose>
-      <topic>lidar</topic>
+      <topic>${ns}/lidar</topic>
       <update_rate>10</update_rate>
       <ray>
         <scan>
           <horizontal>
-            <!-- 3600 samples = 0.1 deg. Needed so adjacent rays stay within one
-                 0.003125m map cell out to ~1.8m; 640 only covered 0.32m. -->
-            <samples>3600</samples>
+            <samples>$(arg lidar_samples)</samples>
             <resolution>1</resolution>
             <min_angle>-3.141593</min_angle>
@@ -49,5 +51,4 @@
         </scan>
         <range>
-          <!-- <min>0.08</min> -->
           <min>0.1</min>
           <max>10.0</max>
@@ -57,8 +58,5 @@
       <always_on>1</always_on>
       <visualize>true</visualize>
-      <gz_frame_id>lidar_link</gz_frame_id>
-      <plugin filename="gz-sim-sensors-system" name="gz::sim::systems::Sensors">
-        <render_engine>ogre2</render_engine>
-      </plugin>
+      <gz_frame_id>${prefix}lidar_link</gz_frame_id>
     </sensor>
   </gazebo>

File: src/nav2_mobile_robot/urdf/nav2_mobile_robot.xacro (robot description, xacro)
@@ -2,4 +2,11 @@
 <robot name="nav_robot"
   xmlns:xacro="http://ros.org/wiki/xacro">
+  <!-- Multi-robot support: every link, joint, TF frame and Gazebo topic is
+       prefixed so N robots can coexist in one /tf tree and one DDS graph.
+       Single robot (both empty) reproduces the original names exactly. -->
+  <xacro:arg name="prefix" default="" />
+  <xacro:arg name="ns" default="" />
+  <xacro:property name="prefix" value="$(arg prefix)" />
+  <xacro:property name="ns" value="$(arg ns)" />
   <xacro:property name="base_radius" value="0.15" />
   <xacro:property name="passive_wheel_height" value="0.04" />
@@ -13,5 +20,5 @@
   <xacro:include filename="lidar.xacro" />
   <!-- <xacro:include filename="ros2_control.xacro" /> -->
-  <link name="base_link">
+  <link name="${prefix}base_link">
     <inertial>
       <inertia ixx="1.0" ixy="0.0" ixz="0.0" iyy="1.0" iyz="0.0" izz="1.0"/>
@@ -34,17 +41,17 @@
     </collision>
   </link>
-  <xacro:passive_wheel_joint name="passive_wheel_front_joint" parent="base_link" child="passive_wheel_front_link">
+  <xacro:passive_wheel_joint name="${prefix}passive_wheel_front_joint" parent="${prefix}base_link" child="${prefix}passive_wheel_front_link">
     <origin xyz="0.115 0.0 0.007" rpy="${-PI/2} 0 0"/>
   </xacro:passive_wheel_joint>
-  <xacro:passive_wheel_link name="passive_wheel_front_link">
+  <xacro:passive_wheel_link name="${prefix}passive_wheel_front_link">
     <origin xyz="0 0.02 0" rpy="${PI/2} 0 0" />
   </xacro:passive_wheel_link>
-  <xacro:passive_wheel_joint name="passive_wheel_back_joint" parent="base_link" child="passive_wheel_back_link">
+  <xacro:passive_wheel_joint name="${prefix}passive_wheel_back_joint" parent="${prefix}base_link" child="${prefix}passive_wheel_back_link">
     <origin xyz="-0.135 0.0 0.009" rpy="${-PI/2} 0 0"/>
   </xacro:passive_wheel_joint>
-  <xacro:passive_wheel_link name="passive_wheel_back_link">
+  <xacro:passive_wheel_link name="${prefix}passive_wheel_back_link">
     <origin xyz="0.02 0.02 0 " rpy="${PI/2} 0 0" />
   </xacro:passive_wheel_link>
-  <xacro:wheel side="right" parent="base_link" translateX="0" translateY="-${base_radius}"/>
-  <xacro:wheel side="left" parent="base_link" translateX="0" translateY="${base_radius}" />
+  <xacro:wheel side="right" parent="${prefix}base_link" translateX="0" translateY="-${base_radius}"/>
+  <xacro:wheel side="left" parent="${prefix}base_link" translateX="0" translateY="${base_radius}" />
 </robot>

File: src/nav2_mobile_robot/urdf/nav2_mobile_robot_macro.xacro (robot description, xacro)
@@ -42,5 +42,5 @@
   </xacro:macro>
   <xacro:macro name="wheel" params="side parent translateX translateY">
-    <link name="${side}_wheel">
+    <link name="${prefix}${side}_wheel">
       <visual>
         <origin xyz="0 0 0" rpy="${PI/2} 0 0 " />
@@ -62,7 +62,7 @@
       </inertial>
     </link>
-    <joint name="${side}_wheel_joint" type="continuous">
+    <joint name="${prefix}${side}_wheel_joint" type="continuous">
       <parent link="${parent}"/>
-      <child link="${side}_wheel"/>
+      <child link="${prefix}${side}_wheel"/>
       <origin xyz="0 ${translateY} 0" rpy="0 0 0" />
       <axis xyz="0 1 0" rpy="0 0 0" />

File: src/nav2_mobile_robot/urdf/odom_plugin.xacro (robot description, xacro)
@@ -6,8 +6,8 @@
       <dimensions>3</dimensions>
       <odom_publish_frequency>50</odom_publish_frequency>
-      <odom_topic>/odom</odom_topic>
-      <odom_frame>odom</odom_frame>
-      <robot_base_frame>base_link</robot_base_frame>
-      <tf_topic>/odom/tf</tf_topic>
+      <odom_topic>${ns}/odom</odom_topic>
+      <odom_frame>${prefix}odom</odom_frame>
+      <robot_base_frame>${prefix}base_link</robot_base_frame>
+      <tf_topic>${ns}/odom/tf</tf_topic>
     </plugin>
   </gazebo>
